File: Storage.kicad_sch (KiCad schematic)
At the start: 3 parts

Commit message: Revision
Changed lines of the file:
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@@
 	(wire
 		(pts
-			(xy 88.9 123.19) (xy 88.9 106.68)
+			(xy 88.9 128.27) (xy 88.9 106.68)
 		)
 		(stroke
@@
 	(symbol
 		(lib_id "power:GND")
-		(at 88.9 123.19 0)
+		(at 88.9 128.27 0)
 		(unit 1)
 		(exclude_from_sim no)
@@
 		(dnp no)
 		(property "Reference" "#PWR018"
-			(at 88.9 129.54 0)
+			(at 88.9 134.62 0)
 			(effects
 				(font
@@
 		)
 		(property "Value" "GND"
+			(at 88.9 133.35 0)
+			(effects
+				(font
+					(size 1.27 1.27)
+				)
+			)
+		)
+		(property "Footprint" ""
 			(at 88.9 128.27 0)
 			(effects
@@
 					(size 1.27 1.27)
 				)
-			)
-		)
-		(property "Footprint" ""
-			(at 88.9 123.19 0)
-			(effects
-				(font
-					(size 1.27 1.27)
-				)
 				(hide yes)
 			)
 		)
 		(property "Datasheet" ""
-			(at 88.9 123.19 0)
+			(at 88.9 128.27 0)
 			(effects
 				(font
@@
 		)
 		(property "Description" "Power symbol creates a global label with name \"GND\" , ground"
-			(at 88.9 123.19 0)
-			(effects
-				(font
+			(at 88.9 128.27 0)
+			(effects
+				(font
