File: USB_C_PORT.kicad_sch (KiCad schematic)
At the start: 6 parts

Commit message: Revision
Parts:
- removed D2, D3: SMF6V0A-E3-08, Diode_SMD:D_SMF, symbol Diode:SMF6V0A
- removed D4: SMF6V0A-E3-08, Diode_SMD:D_SMF, symbol Diode:SMF6V5A
- added U2: USBLC6-2SC6, Package_TO_SOT_SMD:SOT-23-6, symbol Power_Protection:USBLC6-2SC6
Connections:
- net +5V: now also U2.5 (VBUS)
- net GND: now also U2.2 (GND)
- net USB_D+: now also U2.3 (I/O2); no longer PowerUpload1.A6 (D+), PowerUpload1.B6 (D+)
- net USB_D-: now also U2.1 (I/O1); no longer PowerUpload1.A7 (D-), PowerUpload1.B7 (D-)
- new net: PowerUpload1.A6 (D+), PowerUpload1.B6 (D+), U2.4 (I/O2)
- new net: PowerUpload1.A7 (D-), PowerUpload1.B7 (D-), U2.6 (I/O1)
