File: Experimental.kicad_sch (KiCad schematic)
At the start: 65 parts, among them J1 MX128-5.0-04P-GN01-Cu-Y-A, J10 Screw_Terminal, J2 Screw_Terminal, J3 MX128-5.0-04P-GN01-Cu-Y-A, J4 MX128-5.0-04P-GN01-Cu-Y-A, J5 LIPO PIN, J7 MX128-5.0-04P-GN01-Cu-Y-A, J7CHECK 20279-001E-03, J9 MX128-5.0-04P-GN01-Cu-Y-A, P2 LP5907MFX-3.3, Q1 AO3400A, Q2 AO3400A, Q3 AO3400A, U1 NEO-M8N, U2 USBLC6-2SC6

Commit message: Schematic Revision v4
Parts:
- added C12: 100nf, Capacitor_SMD:C_0402_1005Metric, symbol MCASE168SB7105MTNA01:MCASE168SB7105MTNA01
- added C13: 100nF, Capacitor:CAPC1608X90N, symbol MCASE168SB7105MTNA01:MCASE168SB7105MTNA01
- added C14: 10uF, Capacitor_SMD:C_0402_1005Metric, symbol MCASE168SB7105MTNA01:MCASE168SB7105MTNA01
- added Q4: FDN340P, Package_TO_SOT_SMD:SOT-23, symbol Transistor_FET:FDN340P
- added R24, R26, R27, R28: 10k, Resistor:R0402, symbol Device:R_Small
- added R25: 2200, Resistor:R0402, symbol Device:R_Small
- gave numbers to parts that had none: 1
- renumbered C11_47uF to C11_47uF1, C12_47uF to C12_47uF1, GREEN_LED to GREEN_LED1, J7CHECK to J7CHECK1, R to R23
Connections:
- net +3V3: now also C12.2, C13.2, C14.2, R26.1, R27.1, R28.2
- net +7.4V: now also Q4.2 (S), R24.2; no longer Q3.3 (D)
- net GND: now also Q1.2 (S), Q2.2 (S), Q3.2 (S), C12.1, C13.1, C14.1; no longer Q1.3 (D), Q2.3 (D)
- net at J10.1 (Pin_1), J2.1 (Pin_1), R22.2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: now also R14.2, R4.2
- net at ESP32S3.23 (IO21), SDCard1.2 (DAT3/CD): now also R28.1
- net at ESP32S3.28 (IO35), SDCard1.3 (CMD): now also R26.2
- net at ESP32S3.29 (IO36), SDCard1.7 (DAT0): now also R27.2
- net at R20.2, R23.2: now also Q4.3 (D); no longer Q3.2 (S)
- new net: Q4.1 (G), R24.1, R25.2
- new net: Q3.3 (D), R25.1
- new net: J10.2 (Pin_2), Q1.3 (D)
- new net: J2.2 (Pin_2), Q2.3 (D)
Other:
- moved on the sheet: C1, D2, J10, J2, Q1, Q2, R14, R16, R19, R20, R22, R23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

Commit message: Version 4.0
Schematic Cleanup and PCB Layout/Impletementation
Parts:
- removed C11_47uF1: GRM188R60J476ME15D, Capacitor:EEEHP1H4R7P, symbol MCASE168SB7105MTNA01:MCASE168SB7105MTNA01
- removed J4: MX128-5.0-04P-GN01-Cu-Y-A, TerminalBlock:TerminalBlock_MaiXu_MX126-5.0-04P_1x04_P5.00mm, symbol Connector:Screw_Terminal_01x04
- removed R13: 10k, Resistor:R0402, symbol Device:R_Small
- added C12_47uF2: 06034W476MAT2A, Capacitor_SMD:C_0201_0603Metric, symbol MCASE168SB7105MTNA01:MCASE168SB7105MTNA01
- added R29, R30, R31: 10k, Resistor:R0402, symbol Device:R_Small
- C12_47uF1: value GRM188R60J476ME15D -> 06034W476MAT2A; footprint Capacitor:CAPC1608X100N -> Capacitor_SMD:C_0201_0603Metric
- R14, R4: value 2200 -> 10k
Connections:
- net +3V3: now also R27.2, R29.2, R30.2, R31.2; no longer R27.1
- net +5V: now also C12_47uF2.2
- net GND: now also SDCard1.9 (DET_B), C12_47uF2.1
- net at ESP32S3.29 (IO36), SDCard1.7 (DAT0): now also R27.1; no longer R27.2
- net at J10.1 (Pin_1), J2.1 (Pin_1), R22.2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: no longer R14.2, R4.2
- net CS_FLASH: now reaches WSON-8-Flash1.1 (~{CS})
- net CS_FLASH: now also ESP32S3.35 (IO42)
- net DET_A: now reaches ESP32S3.26 (IO45)
- net DET_A: now also SDCard1.10 (DET_A), R30.1
- net at SDCard1.1 (DAT2): now also R31.1
- net at SDCard1.8 (DAT1): now also R29.1
- net at J10.2 (Pin_2), Q1.3 (D): now also R4.2
- net at J2.2 (Pin_2), Q2.3 (D): now also R14.2
- no-connect marks 23 -> 21
Other:
- moved on the sheet: C1, R14, R26, R27, R28, R4

Commit message: Version 5.0!
Parts:
- removed J1, J3, J7, J9: MX128-5.0-04P-GN01-Cu-Y-A, TerminalBlock:TerminalBlock_MaiXu_MX126-5.0-04P_1x04_P5.00mm, symbol Connector:Screw_Terminal_01x04
- removed J10, J2: Screw_Terminal, TerminalBlock:TerminalBlock_MaiXu_MX126-5.0-02P_1x02_P5.00mm, symbol Connector:Screw_Terminal_01x02
- removed P2: LP5907MFX-3.3, Package_TO_SOT_SMD:SOT-23-5, symbol Regulator_Linear:LP5907MFX-3.3
- added C15: 100nF, Capacitor:CAPC1608X90N, symbol MCASE168SB7105MTNA01:MCASE168SB7105MTNA01
- added C16, C17, C18: 10uF, Capacitor_SMD:C_0402_1005Metric, symbol MCASE168SB7105MTNA01:MCASE168SB7105MTNA01
- added C19, C20: 1uf, Capacitor_SMD:C_0402_1005Metric, symbol MCASE168SB7105MTNA01:MCASE168SB7105MTNA01
- added C21: 10nF, Capacitor:CAPC1608X90N, symbol MCASE168SB7105MTNA01:MCASE168SB7105MTNA01
- added D3: B220, Diode_SMD:D_SMB, symbol Diode:B220
- added J1, J2, J3: SPRING_CONN, 6P_SMD_SPRING_CONN, symbol 6P_SMD_SPRING_CONN:1771130
- added L1: 27 nH, Inductor_SMD:L_0402_1005Metric, symbol Device:L
- added NCD0603R2: RED_LED, LED_SMD:LED_0603_1608Metric, symbol Device:LED
- added Q5: AO3400A, Package_TO_SOT_SMD:SOT-23, symbol Transistor_FET:AO3400A
- added R13, R32: 30, Resistor:R0402, symbol Device:R_Small
- added R33: 1k, Resistor:R0402, symbol Device:R_Small
- added R34: 330, Resistor:R0402, symbol Device:R_Small
- added R35, R36: 10k, Resistor:R0402, symbol Device:R_Small
- added R37: 10, Resistor:R0402, symbol Device:R_Small
- added U3: R-783.3-1.0, Converter_DCDC:Converter_DCDC_RECOM_R-78E-0.5_THT, symbol Regulator_Switching:R-783.3-1.0
- C13, C3, C4, C5, C7, C8, C9: Check_prices https://www.snapeda.com/parts/MCASE168SB7105MTNA01/Taiyo+Yu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 -> (none); Description_1 1uF 16V 20% Multilayer Ceramic Capacitor X7R 0603 (1608 Met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 -> SMD/SMT 963-MSAYL21GSSD104KT RPLCMT PN 10V 0.1uF 0805 10%; MAXIMUM_PACKAGE_HEIGHT 0.9mm -> (none); MF Taiyo Yuden -> TAIYO YUDEN; MP MCASE168SB7105MTNA01 -> 963-LMK212SD104KG-T; PARTREV NA -> (none); Package 0603-2 TAIYO -> (none); Price None -> (none); STANDARD IPC-7351B -> (none); SnapEDA_Link https://www.snapeda.com/parts/MCASE168SB7105MTNA01/Taiyo+Yu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 -> (none)
- C14: Availability In Stock -> (none); Check_prices https://www.snapeda.com/parts/MCASE168SB7105MTNA01/Taiyo+Yu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 -> (none); Description_1 1uF 16V 20% Multilayer Ceramic Capacitor X7R 0603 (1608 Met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 -> CL05A106MP5NUNC; Link (none) -> https://www.digikey.com/en/products/detail/samsung-electro-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; MANUFACTURER Taiyo Yuden -> (none); MAXIMUM_PACKAGE_HEIGHT 0.9mm -> (none); MF Taiyo Yuden -> Samsung Electro-Mechanics; MP MCASE168SB7105MTNA01 -> (none); PARTREV NA -> (none); Package 0603-2 TAIYO -> 0402 (1005 Metric); Price None -> $0.08; STANDARD IPC-7351B -> (none); SnapEDA_Link https://www.snapeda.com/parts/MCASE168SB7105MTNA01/Taiyo+Yu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 -> (none)
- NCD0603R1: value RED_LED -> GREEN_LED
- R7: value 5.4k -> 1k; footprint Resistor_SMD:R_0402_1005Metric -> Resistor:R0402
- R8: value 5.4k -> 330; footprint Resistor_SMD:R_0402_1005Metric -> Resistor:R0402
- renumbered GREEN_LED1 to BLUE_LED1
Connections:
- net +3V3: now also C8.2, C9.2, C15.2, C16.2, C18.2, C20.2, J2.1, J2.3, J2.5, U3.3 (OUT); no longer C8.1, C9.1
- net +5V: now also Boot2.2 (B); no longer C2.2, PowerUpload1.A4 (VBUS), PowerUpload1.A9 (VBUS), PowerUpload1.B4 (VBUS), PowerUpload1.B9 (VBUS), U2.5 (VBUS)
- net CHARGE_PYRO: now also ESP32S3.24 (IO47); no longer ESP32S3.20 (IO12)
- net DET_A: now also ESP32S3.14 (IO20); no longer ESP32S3.26 (IO45)
- net GND: now also C3.1, C8.1, C9.1, C15.1, C16.1, C17.1, C18.1, C19.1, C20.1, C21.1, J2.2, J2.4, J2.6, NCD0603R2.1 (K), Q5.2 (S), R36.1, U3.2 (GND); no longer Boot2.1 (A), C3.2, C8.2, C9.2, ESP32S3.17 (IO9), ESP32S3.19 (IO11), R14.1, R4.1
- net PYRO2_FIRE: now also ESP32S3.21 (IO13), R19.1; no longer ESP32S3.12 (IO8), R18.1
- net ~{RESET}: now also ESP32S3.35 (IO42); no longer ESP32S3.39 (IO1)
- net at R27.1, SDCard1.7 (DAT0): now also ESP32S3.13 (IO19); no longer ESP32S3.29 (IO36)
- net at R22.2, R23.1: now also J3.2, J3.4, J3.6
- net Pad_8: now reaches ESP32S3.8 (IO15)
- net Pad_8: now also J1.6
- net D+: now reaches ESP32S3.9 (IO16)
- net D+: now also U2.3 (I/O2)
- net D-: now reaches ESP32S3.10 (IO17)
- net D-: now also U2.1 (I/O1)
- net at ESP32S3.11 (IO18): now also R28.1, SDCard1.2 (DAT3/CD)
- net at WSON-8-Flash1.2 (DO/IO_{1}): now also ESP32S3.30 (IO37); no longer ESP32S3.32 (IO39)
- net at WSON-8-Flash1.3 (~{WP}/IO_{2}): now also ESP32S3.31 (IO38); no longer ESP32S3.33 (IO40)
- net at WSON-8-Flash1.5 (DI/IO_{0}): now also ESP32S3.32 (IO39); no longer ESP32S3.31 (IO38)
- net CLK: now reaches SDCard1.5 (CLK), WSON-8-Flash1.6 (CLK)
- net CLK: now also ESP32S3.28 (IO35); no longer ESP32S3.30 (IO37)
- net at WSON-8-Flash1.7 (~{HOLD}/~{RESET}/IO_{3}): now also ESP32S3.33 (IO40); no longer ESP32S3.34 (IO41)
- net at ESP32S3.15 (IO3): now also J1.1; no longer U1.3 (TIMEPULSE)
- net SCL: now reaches ESP32S3.16 (IO46)
- net SCL: now also Barometer1.2 (SCK), IMU6axis1.13 (SCL), Magnometer1.1 (SCL/SPC), R3.1
- net SDA: now reaches Barometer1.4 (SDI), IMU6axis1.14 (SDA), Magnometer1.11 (SDA/SDI/SDO), R6.1
- net SDA: now also ESP32S3.17 (IO9); no longer ESP32S3.21 (IO13)
- net at ESP32S3.25 (IO48): no longer R7.1
- net Pad12_CMD: now reaches R26.2, SDCard1.3 (CMD)
- net Pad12_CMD: now also ESP32S3.12 (IO8); no longer ESP32S3.28 (IO35)
- net at Boot2.3 (C): now also R33.1; no longer ESP32S3.3 (EN)
- net at ESP32S3.36 (RXD0): now also R13.1; no longer U1.20 (TXD/SPI_MISO)
- net at ESP32S3.37 (TXD0): now also R32.1; no longer U1.21 (RXD/SPI_MOSI)
- net at ESP32S3.38 (IO2): now also U1.3 (TIMEPULSE); no longer U1.14 (LNA_EN)
- net at ESP32S3.4 (IO4): now also J1.2
- net at ESP32S3.5 (IO5): now also J1.3
- net at ESP32S3.6 (IO6): now also J1.4
- net at ESP32S3.7 (IO7): now also J1.5
- net at Q1.3 (D), R4.2: now also J3.5
- net at J7CHECK1.1, U1.11 (RF_IN): now also L1.2
- net at Magnometer1.4 (C1): now also C3.2; no longer C3.1
- net at Q2.3 (D), R14.2: now also J3.3
- net at U1.9 (VCC_RF): now also R37.1
- net at R17.1: now also ESP32S3.3 (EN), C17.2, C19.2; no longer Boot2.2 (B)
- net CS_FLASH: no longer names the net of WSON-8-Flash1.1 (~{CS})
- net CS_FLASH: now also ESP32S3.29 (IO36); no longer ESP32S3.35 (IO42)
- net PYRO_FIRE renamed PYRO1_CONTINUITY
- net PYRO1_CONTINUITY: now also R35.1; no longer R19.1
- new net: J3.1, Q5.3 (D), R35.2
- new net: C21.2, L1.1, R37.2
- new net: NCD0603R2.2 (A), R33.2
- new net: ESP32S3.26 (IO45), R7.1
- new net: ESP32S3.39 (IO1), U1.14 (LNA_EN)
- new net: Boot2.1 (A), C2.2, D3.1 (K), U2.5 (VBUS), U3.1 (IN)
- new net: D3.2 (A), PowerUpload1.A4 (VBUS), PowerUpload1.A9 (VBUS), PowerUpload1.B4 (VBUS), PowerUpload1.B9 (VBUS)
- new net: Q5.1 (G), R34.2, R36.2
- new net: R13.2, U1.20 (TXD/SPI_MISO)
- new net: R32.2, U1.21 (RXD/SPI_MOSI)
- new net PYRO1_FIRE: ESP32S3.19 (IO11), R34.1
- new net PYRO2_CONTINUITY: ESP32S3.20 (IO12), R14.1
- new net PYRO3_CONTINUITY: ESP32S3.22 (IO14), R4.1
- new net PYRO3_FIRE: ESP32S3.23 (IO21), R18.1
- no-connect marks 21 -> 20
Other:
- note added: "Toggle power... resister to prevent short."
- moved on the sheet: BLUE_LED1, C1, D2, J7CHECK1, Q1, Q2, Q3, Q4, R14, R15, R16, R17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
