File: _autosave-Experimental.kicad_sch (KiCad schematic)
At the start: 65 parts, among them J1 MX128-5.0-04P-GN01-Cu-Y-A, J10 Screw_Terminal, J2 Screw_Terminal, J3 MX128-5.0-04P-GN01-Cu-Y-A, J4 MX128-5.0-04P-GN01-Cu-Y-A, J5 LIPO PIN, J7 MX128-5.0-04P-GN01-Cu-Y-A, J7CHECK 20279-001E-03, J9 MX128-5.0-04P-GN01-Cu-Y-A, P2 LP5907MFX-3.3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

Commit message: update
Parts:
- gave numbers to parts that had none: 1
- renumbered C11_47uF to C11_47uF1, C12_47uF to C12_47uF1, GREEN_LED to GREEN_LED1, J7CHECK to J7CHECK1, R to R23
Changed lines of the file:
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@@
 		(dnp no)
 		(fields_autoplaced yes)
-		(property "Reference" "C12_47uF"
+		(property "Reference" "C12_47uF1"
 			(at 380.238 233.934 90)
 			(effects
@@
 			(project "Experimental"
 				(path "/d685641e-0e6b-462c-92c0-fbf0ccf1a433"
-					(reference "C12_47uF")
+					(reference "C12_47uF1")
 					(unit 1)
 				)
@@
 		(dnp no)
 		(fields_autoplaced yes)
-		(property "Reference" "D?"
+		(property "Reference" "D2"
 			(at 66.04 202.2474 90)
 			(effects
@@
 			(project "Experimental"
 				(path "/d685641e-0e6b-462c-92c0-fbf0ccf1a433"
-					(reference "D?")
+					(reference "D2")
 					(unit 1)
 				)
@@
 		(dnp no)
 		(fields_autoplaced yes)
-		(property "Reference" "J7CHECK"
+		(property "Reference" "J7CHECK1"
 			(at 90.932 43.18 90)
 			(effects
@@
 			(project "Experimental"
 				(path "/d685641e-0e6b-462c-92c0-fbf0ccf1a433"
-					(reference "J7CHECK")
+					(reference "J7CHECK1")
 					(unit 1)
 				)
@@
 		(dnp no)
 		(fields_autoplaced yes)
-		(property "Reference" "C11_47uF"
+		(property "Reference" "C11_47uF1"
 			(at 361.442 234.188 90)
 			(effects
@@
 			(project "Experimental"
 				(path "/d685641e-0e6b-462c-92c0-fbf0ccf1a433"
-					(reference "C11_47uF")
+					(reference "C11_47uF1")
 					(unit 1)
 				)
@@
 		(dnp no)
 		(fields_autoplaced yes)
-		(property "Reference" "R"
+		(property "Reference" "R23"
 			(at 59.69 180.34 90)
 			(effects
@@
 			(project "Experimental"
 				(path "/d685641e-0e6b-462c-92c0-fbf0ccf1a433"
-					(reference "R")
+					(reference "R23")
 					(unit 1)
 				)
@@
 		(dnp no)
 		(fields_autoplaced yes)
-		(property "Reference" "GREEN_LED"
+		(property "Reference" "GREEN_LED1"
 			(at 262.128 181.356 90)
 			(effects
@@
 			(project "Experimental"
 				(path "/d685641e-0e6b-462c-92c0-fbf0ccf1a433"
-					(reference "GREEN_LED")
+					(reference "GREEN_LED1")
 					(unit 1)
 				)
